File: CAPSTONE_BMS/PCB/Switching_PCB/Switching_PCB.kicad_sch (KiCad schematic)
At the start: 10 parts, among them J1 Screw_Terminal_01x02, J2 Screw_Terminal_01x02, Q1 IRF4905, Q2 IRF4905, Q3 2N2219, U1 NUCLEO64-F411RE

Commit message: added schematics and few file changes
Parts:
- removed U1: NUCLEO64-F411RE, Module:ST_Morpho_Connector_144_STLink, symbol MCU_Module:NUCLEO64-F411RE
- added D2: 1N5400, Diode_THT:D_DO-201AD_P15.24mm_Horizontal, symbol Diode:1N5400
- added J3: Screw_Terminal_01x02, symbol Connector:Screw_Terminal_01x02
- added Q4: 2N2219, Package_TO_SOT_THT:TO-39-3, symbol Transistor_BJT:2N2219
- added Q5, Q6: IRF4905, Package_TO_SOT_THT:TO-220-3_Vertical, symbol Transistor_FET:IRF4905
- added R4: 1K, symbol Device:R
- added R5: 100K, symbol Device:R
- added R6: 10K, symbol Device:R
- added U1: NUCLEO-F401RE, NUCLEO-F401RE:ST_NUCLEO-F401RE, symbol NUCLEO-F401RE:NUCLEO-F401RE
- added U2, U3: INA260, Package_SO:TSSOP-16_4.4x5mm_P0.65mm, symbol Sensor:INA260
- added U4: 1.3inch oled, symbol 1.3 Inch I2C OLED Display Module 128×64 4-Pin Blue:1.3inch_SSD1306_OLED_
Connections:
- net 10V is gone; now on net +10V_0: Q1.3 (S), Q2.3 (S)
- net Collector is gone; now on net R3: R3.1
- net Q1_Pin1 is gone; now on net Q1_Pin2: J2.1 (Pin_1)
- net Q3_Base is gone; now on net GND: R1.2, R2.1
- net D1: now also D1.1 (K)
- net GND: now also Q3.1 (E), Q3.2 (B), J3.2 (Pin_2), Q4.1 (E), R5.2, U1.6_6 (GND), U1.6_7 (GND), U2.11 (GND), U2.6 (GND), U3.11 (GND), U3.6 (GND)
- net Gate_Q1: now also Q1.1 (G), Q2.1 (G)
- net PB4: now also U1.10_27 (PB4)
- net R3: no longer Q1.1 (G), Q2.1 (G)
- net +10V renamed +10V_0
- net +10V_0: now also U2.1 (IN+), U2.2 (IN+), U2.3 (IN+); no longer Q2.2 (D)
- net J2_1 renamed Q1_Pin2
- net Q1_Pin2: now also Q5.2 (D)
- removed net R1: D1.1 (K), Q3.2 (B)
- new net +10V_1: J3.1 (Pin_1), Q5.3 (S), Q6.3 (S), U3.1 (IN+), U3.2 (IN+), U3.3 (IN+)
- new net D2: D2.1 (K), R4.1
- new net GND_S1: U1.7_19 (GND_S1), U1.7_20 (GND_S1), U1.7_22 (GND_S1), U1.7_8 (GND_S1)
- new net GND_S2: U1.10_20 (GND_S2), U1.10_9 (GND_S2)
- new net Gate_Q5: Q5.1 (G), Q6.1 (G), R6.2
- new net PB5: D2.2 (A), U1.10_29 (PB5)
- new net Q2_Pin2: Q2.2 (D), U2.14 (IN-), U2.15 (IN-), U2.16 (IN-)
- new net Q6_Pin2: Q6.2 (D), U3.14 (IN-), U3.15 (IN-), U3.16 (IN-)
- new net R4: Q4.2 (B), R4.2, R5.1
- new net R6: Q4.3 (C), R6.1
- new net U1_5V: U1.6_5 (+5V), U2.10 (VS), U3.10 (VS)
Other:
- note removed: "Footprint is same to F446RE,so using this as alternative."
- moved on the sheet: D1, J1, J2, Q1, Q2, Q3, R1, R2, R3
